Commit message: added force sensor in UWsim_scene1.xml

File: simulator_stack/kraken_visualization/kraken/scenes/scene.urdf (robot description, URDF)
Before this commit: robot scene, 11 links, 10 joints
Links:
- removed link gate_marker2
- link pool: mass None -> 0
Joints:
- removed joint gate_marker2_to_pool
